File: esp-32wrover.sch (KiCad schematic (older format))
At the start: 68 parts, among them CON1 BARREL_JACK, P1 Power, P2 Analog, P3 Digital, P4 Digital, P5 CONN_1, P6 CONN_1, P7 CONN_1, P8 CONN_1, P9 CONN_01X04, Q1 12Mhz, Q2 32.768Khz, Q3 Q_NPN_BEC, Q4 Q_NPN_BEC, SW1 SW_PUSH, SW2 SW_PUSH, U1 usb_mini_b, U2 MCP16311-MNY, U3 BD00GA5WEFJ, U4 PL2303HXA, U5 MCP6001R, U6 ESP32-WROVER, U7 IRLM6402

Commit message: tạo khối ADC
Parts:
- added D?: L-TX, symbol LED
- added D?: L-RX, symbol LED
- added D? (x6): ZENER_3.3V, symbol ZENER
- added R? (x2): 470R, 0603_N, symbol R
- added R? (x6): 220k/1%, 0603_N, symbol R
- added R? (x6): 100k, 0603_N, symbol R
Connections:
- net +3V3: now also R?.1, R?.1
- net ADC-0: now also R?.1, R?.2
- net ADC-1: now also R?.1, R?.2
- net ADC-2: now also R?.1, R?.2
- net ADC-3: now also R?.1, R?.2
- net ADC-4: now also R?.1, R?.2
- net ADC-5: now also R?.1, R?.2
- net RXD: now also D?.1 (K)
- net TXD: now also D?.1 (K)
- net A0: now reaches P2.1
- net A0: now also D?.1 (K), R?.1
- net A1: now reaches P2.2
- net A1: now also D?.1 (K), R?.1
- net A2: now reaches P2.3
- net A2: now also D?.1 (K), R?.1
- net A4: now reaches P2.4
- net A4: now also D?.1 (K), R?.1
- net A5: now reaches P2.5
- net A5: now also D?.1 (K), R?.1
- net A6: now reaches P2.6
- new net: D?.2 (A), R?.2 (x8)
- new net A3: D?.1 (K), R?.1
- no-connect marks 18 -> 10
Other:
- note added: "1 1 1 1\n 0 0 1 1\n 1 0 0 1\n 0 1 1 0"
- note added: "ADC"
- note added: "Auto program circuit\n"
- note added: "BUTTON"
- note added: "DTR"
- note added: "ESP-32 WROVER"
- note added: "GPIO0"
- note added: "HEADER-OLED"
- note added: "POWER-SOURCE"
- note added: "RST"
- note added: "RTS"
- note added: "USB-UART"
- note added: "WIFI-UNO-32S"
- note removed: "Shield for Arduino that uses\nthe same pin disposition\nlike "Uno" board Rev 3."
- moved on the sheet: C19, C20, C5, C7, C8, Q1, Q3, Q4, R13, R14, R15, R19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

Commit message: nối IO
Connections:
- net GPIO0: now also P4.3 (P3)
- net GPIO2: now also P4.4 (P4)
- net RXD: now also P4.1 (P1)
- net TXD: now also P4.2 (P2)
- net IO12: now reaches P4.5 (P5)
- net IO13: now reaches P4.6 (P6)
- net IO14: now reaches P4.7 (P7)
- net IO15: now reaches P4.8 (P8)
- net CMD: now reaches P3.1 (P1)
- net IO27: now reaches P3.10 (P10)
- net CLK: now reaches P3.2 (P2)
- net SDO: now reaches P3.3 (P3)
- net SD1: now reaches P3.5 (P5)
- net SD2: now reaches P3.6 (P6)
- net SD3: now reaches P3.7 (P7)
- net IO17: now reaches P3.8 (P8)
- net IO16: now reaches P3.9 (P9)
Changed lines of the file:
@@
 Wire Wire Line
 	14145 2925 14175 2925
+Text GLabel 7355 3655 0    39   Input ~ 0
+IO27
+Text GLabel 7355 3750 0    39   Input ~ 0
+IO14
+Text GLabel 7355 3850 0    39   Input ~ 0
+IO12
+Text GLabel 9460 2520 2    39   Input ~ 0
+IO23
+Text GLabel 9480 2620 2    39   Input ~ 0
+IO22
+Text GLabel 9470 2915 2    39   Input ~ 0
+IO21
+Text GLabel 9460 3115 2    39   Input ~ 0
+IO27
+Text GLabel 9440 3210 2    39   Input ~ 0
+IO18
+Text GLabel 9430 3415 2    39   Input ~ 0
+IO17
+Text GLabel 9430 3510 2    39   Input ~ 0
+IO16
+Text GLabel 8110 4380 3    39   Input ~ 0
+IO13
+Text GLabel 8210 4380 3    39   Input ~ 0
+SD2
+Text GLabel 8305 4380 3    39   Input ~ 0
+SD3
+Text GLabel 8405 4380 3    39   Input ~ 0
+CMD
+Text GLabel 8505 4385 3    39   Input ~ 0
+CLK
+Text GLabel 8610 4380 3    39   Input ~ 0
+SDO
+Text GLabel 8715 4385 3    39   Input ~ 0
+SD1
+Text GLabel 8810 4390 3    39   Input ~ 0
+IO15
+Text GLabel 15275 2325 2    39   Input ~ 0
+TXD
+Text GLabel 15280 2225 2    39   Input ~ 0
+RXD
+Text GLabel 15280 2620 2    39   Input ~ 0
+IO12
+Text GLabel 15280 2825 2    39   Input ~ 0
+IO14
+Text GLabel 15305 2025 2    39   Input ~ 0
+IO27
+Text GLabel 15330 1825 2    39   Input ~ 0
+IO17
+Text GLabel 15305 1925 2    39   Input ~ 0
+IO16
+Text GLabel 15275 2425 2    39   Input ~ 8
+GPIO0
+Text GLabel 15270 2525 2    39   Input ~ 0
+GPIO2
+Text GLabel 15285 2925 2    39   Input ~ 0
+IO15
+Text GLabel 15330 1625 2    39   Input ~ 0
+SD2
+Text GLabel 15280 2725 2    39   Input ~ 0
+IO13
+Text GLabel 15365 1725 2    39   Input ~ 0
+SD3
+Text GLabel 15340 1125 2    39   Input ~ 0
+CMD
+Text GLabel 15350 1225 2    39   Input ~ 0
+CLK
+Text GLabel 15345 1325 2    39   Input ~ 0
+SDO
+Text GLabel 15350 1525 2    39   Input ~ 0
+SD1
+Wire Wire Line
+	15340 1125 15200 1125
+Wire Wire Line
+	15350 1225 15200 1225
+Wire Wire Line
+	15345 1325 15200 1325
+Wire Wire Line
+	15350 1525 15200 1525
+Wire Wire Line
+	15330 1625 15200 1625
+Wire Wire Line
+	15365 1725 15200 1725
+Wire Wire Line
+	15330 1825 15200 1825
+Wire Wire Line
+	15305 1925 15200 1925
+Wire Wire Line
+	15305 2025 15200 2025
+Wire Wire Line
+	15280 2225 15200 2225
+Wire Wire Line
+	15275 2325 15200 2325
+Wire Wire Line
+	15200 2425 15275 2425
+Wire Wire Line
+	15270 2525 15200 2525
+Wire Wire Line
+	15280 2620 15280 2625
+Wire Wire Line
+	15280 2625 15200 2625
+Wire Wire Line
+	15280 2725 15200 2725
+Wire Wire Line
+	15280 2825 15200 2825
+Wire Wire Line
+	15285 2925 15200 2925
 $EndSCHEMATC

Commit message: noi io
Connections:
- net CLK: now also U6.20 (CLK)
- net CMD: now also U6.19 (CMD)
- net IO12: now also U6.14 (IO12)
- net IO13: now also U6.16 (IO13)
- net IO14: now also U6.13 (IO14)
- net IO15: now also U6.23 (IO15)
- net IO16: now also U6.27 (IO16)
- net IO17: now also U6.28 (IO17)
- net IO18: now also U6.30 (IO18)
- net IO21: now also U6.33 (IO21)
- net IO22: now also U6.36 (IO22)
- net IO23: now also U6.37 (IO23)
- net IO27: now also U6.12 (IO27), U6.31 (IO19)
- net SD1: now also U6.22 (SD1)
- net SD2: now also U6.17 (SD2)
- net SD3: now also U6.18 (SD3)
- net SDO: now also U6.21 (SDO)
Changed lines of the file:
@@
 Wire Wire Line
 	14145 2925 14175 2925
-Text GLabel 7355 3655 0    39   Input ~ 0
+Text GLabel 7355 3665 0    39   Input ~ 0
 IO27
-Text GLabel 7355 3750 0    39   Input ~ 0
+Text GLabel 7345 3765 0    39   Input ~ 0
 IO14
-Text GLabel 7355 3850 0    39   Input ~ 0
+Text GLabel 7355 3865 0    39   Input ~ 0
 IO12
-Text GLabel 9460 2520 2    39   Input ~ 0
+Text GLabel 9460 2515 2    39   Input ~ 0
 IO23
-Text GLabel 9480 2620 2    39   Input ~ 0
+Text GLabel 9480 2610 2    39   Input ~ 0
 IO22
 Text GLabel 9470 2915 2    39   Input ~ 0
@@
 Text GLabel 9460 3115 2    39   Input ~ 0
 IO27
-Text GLabel 9440 3210 2    39   Input ~ 0
+Text GLabel 9445 3215 2    39   Input ~ 0
 IO18
 Text GLabel 9430 3415 2    39   Input ~ 0
 IO17
-Text GLabel 9430 3510 2    39   Input ~ 0
+Text GLabel 9420 3515 2    39   Input ~ 0
 IO16
 Text GLabel 8110 4380 3    39   Input ~ 0
@@
 Text GLabel 8210 4380 3    39   Input ~ 0
 SD2
-Text GLabel 8305 4380 3    39   Input ~ 0
+Text GLabel 8310 4380 3    39   Input ~ 0
 SD3
-Text GLabel 8405 4380 3    39   Input ~ 0
+Text GLabel 8410 4380 3    39   Input ~ 0
 CMD
-Text GLabel 8505 4385 3    39   Input ~ 0
+Text GLabel 8510 4385 3    39   Input ~ 0
 CLK
 Text GLabel 8610 4380 3    39   Input ~ 0
 SDO
-Text GLabel 8715 4385 3    39   Input ~ 0
+Text GLabel 8710 4390 3    39   Input ~ 0
 SD1
 Text GLabel 8810 4390 3    39   Input ~ 0
@@
 Wire Wire Line
 	15285 2925 15200 2925
+Wire Wire Line
+	7355 3665 7510 3665
+Wire Wire Line
+	7345 3765 7510 3765
+Wire Wire Line
+	7355 3865 7510 3865
+Wire Wire Line
+	8110 4315 8110 4380
+Wire Wire Line
+	8210 4315 8210 4380
+Wire Wire Line
+	8310 4315 8310 4380
+Wire Wire Line
+	8410 4315 8410 4380
+Wire Wire Line
+	8510 4315 8510 4385
+Wire Wire Line
+	8610 4315 8610 4380
+Wire Wire Line
+	8710 4315 8710 4390
+Wire Wire Line
+	8810 4315 8810 4390
+Wire Wire Line
+	9420 3515 9360 3515
+Wire Wire Line
+	9430 3415 9360 3415
+Wire Wire Line
+	9445 3215 9360 3215
+Wire Wire Line
+	9460 3115 9360 3115
+Wire Wire Line
+	9470 2915 9360 2915
+Wire Wire Line
+	9480 2610 9410 2610
+Wire Wire Line
+	9410 2610 9410 2615
+Wire Wire Line
+	9410 2615 9360 2615
+Wire Wire Line
+	9460 2515 9360 2515
 $EndSCHEMATC
