File: esp-32wrover.kicad_pcb (KiCad board)
At the start: 2 copper layers, 68.6 x 53.3 mm, 81 parts, among them CON1 BARREL_JACK, P1 CONN_01X04, P10 CONN_1, P2 ICSP, P3 Analog, P4 Analog, P5 Digital, P6 Digital, P7 CONN_1, P8 CONN_1, P9 CONN_1, Q1 Q_NPN_BEC, Q2 Q_NPN_BEC, SW1 SW_PUSH, SW2 SW_PUSH, U1 usb_mini_b, U2 MCP16311-MNY, U3 PL2303HXA, U4 BD00GA5WEFJ, U5 MCP6001R, U6 ESP32-WROVER, U7 IRLM6402, X1 CRYSTAL_ABM3C, Y1 32.768Khz

Commit message: cap nhat 3d cho pcb
Parts:
- added G***: LOGO, new:logo-iotmakervn_7-5x5, F.Cu at (147.5, 91.4)
- added G***: LOGO, new:logo_openhardware_5x5mm, F.Cu at (155.5, 91.3)
- added G***: LOGO, new:logo_cc-bby-sa_14-1x5mm, B.Cu at (176.1, 105.2)
- added G***: LOGO, new:RST, F.Cu at (115.8, 77.9)
- added G***: LOGO, new:logo-jack_7.4x3, F.Cu at (115.6, 124.8)
Other:
- board text added: "+3.3V"
- board text added: "+5V"
- board text added: "A0"
- board text added: "A1"
- board text added: "A2"
- board text added: "A3"
- board text added: "A4"
- board text added: "A5"
- board text added: "CLK"
- board text added: "CMD"
- board text added: "GND"
- board text added: "ICSP"
- board text added: "IO0"
- board text added: "IO12"
- board text added: "IO13"
- board text added: "IO14"
- board text added: "IO15"
- board text added: "IO16"
- board text added: "IO17"
- board text added: "IO2"
- board text added: "IO27"
- board text added: "RST"
- board text added: "RX"
- board text added: "SD0"
- board text added: "SD1"
- board text added: "SD2"
- board text added: "SD3"
- board text added: "TX"
- board text added: "Vin"
- board text added: "http://esp8266.vn"
